File: rp2040_jtag_debugger/rp2040_jtag_debugger.kicad_pcb (KiCad board)
At the start: 2 copper layers, 50 x 47.2 mm, 56 parts, among them J1 USB_C_Receptacle_USB2.0, J2 Conn_ARM_JTAG_SWD_20, J3 BOOT, J4 SWD, U1 SIT2001B, U2 W25Q16JVZPIM, U3 RP2040, U4 TCR3UF33ALM

Commit message: wip: fix DRC
Parts:
- removed REF**: OSHW-Logo2_7.3x6mm_SilkScreen, Symbol:OSHW-Logo2_7.3x6mm_SilkScreen
- removed TP4: TestPoint, TestPoint:TestPoint_Pad_D1.0mm
- added TP1: TestPoint, TestPoint:TestPoint_Pad_D1.0mm, F.Cu at (106.8, 82.4)
Connections:
- net +3V3 renamed +3.3V
Routing:
- net +3.3V: track 168.7 -> 158.8 mm
- net GND: track 75.0 -> 79.3 mm

Commit message: wip
Parts:
- moved R14 3.42 mm to (116.5, 85.6), turned to 180 degrees
- moved R13 1.87 mm to (116.5, 84.1), turned to 180 degrees
Routing:
- net GND: track 79.3 -> 68.4 mm, vias 182 -> 176
- net /D+: track 31.4 -> 21.7 mm
- net /D-: track 28.3 -> 20.5 mm
- net /RD+: track 8.10 -> 10.9 mm
- net /RD-: track 8.08 -> 10.2 mm
- net +3.3V: track 158.8 -> 159.3 mm
Other:
- board text added: "PWR ACT"
- board text removed: "PWD ACT"

Commit message: wip
Parts:
- removed RN1: R_Network08, Resistor_THT:R_Array_SIP9
- removed U3: RP2040, rp2040:RP2040_QFN56_HandSolderHack
- added R19: 10k, Resistor_SMD:R_0603_1608Metric, F.Cu at (133.0, 63.7)
- added R20: 10k, Resistor_SMD:R_0603_1608Metric, F.Cu at (133.0, 80.7)
- added R21: 10k, Resistor_SMD:R_0603_1608Metric, F.Cu at (133.0, 72.9)
- added U5: RP2040, rp2040:RP2040_QFN56_HandSolderHack, F.Cu at (120.2, 72.6)
- C10, C4: value 10uF -> 1uF
- R15: value 100k -> 10k
- moved TP1 6.76 mm to (110.9, 87.8)
Routing:
- net GND: track 68.4 -> 45.6 mm, vias 176 -> 154
- net +3.3V: track 159.3 -> 173.8 mm, vias 14 -> 16
- net Net-(J1-CC2): track 9.33 -> 12.3 mm
- net Net-(U1-OE): track 5.99 -> 4.12 mm, vias 0 -> 2
- added copper zone on B.Cu, net +3.3V
Other:
- board text added: "RP2040 JTAG debugger version 2023/04/10 @tnishinaga"
- board text removed: "RP2040 JTAG debugger version 2022/09/13 @tnishinaga"

Commit message: v2023.07.27
Parts:
- C3: value 0.1uF -> 1uF
- D2: footprint Diode_SMD:D_SOD-323 -> cuhs20s30:US2H
- U2: value W25Q16JVZPIM -> W25Q16JVSNIQ; footprint Package_SON:WSON-8-1EP_6x5mm_P1.27mm_EP3.4x4.3mm -> Package_SO:SO-8_3.9x4.9mm_P1.27mm
- moved R5 14.9 mm to (104.2, 65.3)
- moved GND 7.28 mm to (103.8, 89.3)
- moved D2 4.40 mm to (109.3, 89.5), turned to 180 degrees
- moved C10 1.97 mm to (106.7, 87.3)
- moved C4 1.96 mm to (106.7, 84.3)
- moved +5V 1.92 mm to (106.8, 81.2)
- moved R16 0.62 mm to (104.2, 81.2)
- renumbered TP3 to +5V, TP1 to GND
Routing:
- net +5V: track 24.9 -> 34.8 mm, vias 0 -> 2
- net +3.3V: track 173.8 -> 178.6 mm
- net Net-(J1-CC2): track 12.3 -> 16.7 mm
- net GND: track 45.6 -> 41.4 mm, vias 154 -> 163
- net /QSPI_SD3: track 14.5 -> 17.5 mm
- net /QSPI_SCLK: track 13.1 -> 16.1 mm
- net /QSPI_SD0: track 11.5 -> 14.4 mm
- net /QSPI_CSN: track 23.5 -> 21.4 mm
- net Net-(U4-EN): track 3.01 -> 4.97 mm
- net +1V1: track 40.1 -> 41.8 mm
- net /QSPI_SD1: track 15.9 -> 17.4 mm
- net /QSPI_SD2: track 14.4 -> 15.8 mm
- net Net-(U5-RUN): track 6.23 -> 7.54 mm
Other:
- board text added: "RP2040 JTAG debugger version 2023/07/27 @tnishinaga"
- board text removed: "RP2040 JTAG debugger version 2023/04/10 @tnishinaga"

Commit message: update to 2023/09/09 version
Parts:
- removed +5V, GND: TestPoint, TestPoint:TestPoint_Pad_D1.0mm
- added TP1: TestPoint, TestPoint:TestPoint_Pad_D1.0mm, F.Cu at (110.8, 87.8)
- added TP3: TestPoint, TestPoint:TestPoint_Pad_D1.0mm, F.Cu at (108.6, 81.6)
- D2: value CUHS20S30 -> RB160M-30TR; footprint cuhs20s30:US2H -> pmdu:D_PMDU
- U2: footprint Package_SO:SO-8_3.9x4.9mm_P1.27mm -> Package_SO:SOIC-8_5.23x5.23mm_P1.27mm
- moved D2 3.86 mm to (108.6, 85.7), turned to 0 degrees
- moved J3 1.91 mm to (135.5, 90.1)
- moved R1 1.70 mm to (133.0, 89.7)
- moved C1 0.98 mm to (123.6, 90.7)
- moved R16 0.43 mm to (104.0, 81.6)
- moved R21 0.09 mm to (132.9, 72.9)
Routing:
- net +5V: track 34.8 -> 26.7 mm, vias 2 -> 0
- net +3.3V: track 178.6 -> 181.8 mm
- net /QSPI_CSN: track 21.4 -> 24.1 mm
- net Net-(U4-EN): track 4.97 -> 3.05 mm
- net GND: track 41.4 -> 39.8 mm, vias 163 -> 157
- net /VO: track 9.65 -> 11.2 mm
- net /QSPI_SD3: track 17.5 -> 18.2 mm
- net /QSPI_SD2: track 15.8 -> 16.5 mm
- net /QSPI_SD0: track 14.4 -> 15.1 mm
- net /QSPI_SD1: track 17.4 -> 18.0 mm
- net /QSPI_SCLK: track 16.1 -> 16.6 mm
Other:
- board text added: "RP2040 JTAG debugger version 2023/09/09 @tnishinaga"
- board text removed: "RP2040 JTAG debugger version 2023/07/27 @tnishinaga"
