File: rp2040_jtag_debugger/rp2040_jtag_debugger.kicad_sch (KiCad schematic)
At the start: 55 parts, among them J1 USB_C_Receptacle_USB2.0, J2 Conn_ARM_JTAG_SWD_20, J3 BOOT, J4 SWD, U1 SIT2001B, U2 W25Q16JVZPIM, U3 RP2040, U4 TCR3UF33ALM

Commit message: wip: fix DRC
Parts:
- U3: footprint Package_DFN_QFN:QFN-56-1EP_7x7mm_P0.4mm_EP5.6x5.6mm -> rp2040:RP2040_QFN56_HandSolderHack
Changed lines of the file:
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@@
       (effects (font (size 1.27 1.27)))
     )
-    (property "Footprint" "Package_DFN_QFN:QFN-56-1EP_7x7mm_P0.4mm_EP5.6x5.6mm" (at 157.48 85.09 0)
+    (property "Footprint" "rp2040:RP2040_QFN56_HandSolderHack" (at 157.48 85.09 0)
       (effects (font (size 1.27 1.27)) hide)
     )

Commit message: wip
Parts:
- removed RN1: R_Network08, Resistor_THT:R_Array_SIP9, symbol Device:R_Network08
- removed U3: RP2040, rp2040:RP2040_QFN56_HandSolderHack, symbol rp2040:RP2040
- added R19, R20, R21: 10k, Resistor_SMD:R_0603_1608Metric, symbol Device:R
- added U5: RP2040, rp2040:RP2040_QFN56_HandSolderHack, symbol MCU_RaspberryPi:RP2040
- C10, C4: value 10uF -> 1uF
- R15: value 100k -> 10k; MPN RC0603FR-10100KL -> ERJ-3EKF1002V
- R16: MPN RK73Z1JTTD -> ERJ-3EKF1002V
Connections:
- net +1V1: now also U5.23 (DVDD), U5.45 (VREG_VOUT), U5.50 (DVDD)
- net +3.3V: now also R19.2, R20.2, U5.1 (IOVDD), U5.10 (IOVDD), U5.22 (IOVDD), U5.33 (IOVDD), U5.42 (IOVDD), U5.43 (ADC_AVDD), U5.44 (VREG_IN), U5.48 (USB_VDD), U5.49 (IOVDD)
- net GND: now also R21.1, U5.19 (TESTEN), U5.57 (GND)
- net LED: now also U5.28 (GPIO17)
- net QSPI_CSN: now also U5.56 (QSPI_SS)
- net QSPI_SCLK: now also U5.52 (QSPI_SCLK)
- net QSPI_SD0: now also U5.53 (QSPI_SD0)
- net QSPI_SD1: now also U5.55 (QSPI_SD1)
- net QSPI_SD2: now also U5.54 (QSPI_SD2)
- net QSPI_SD3: now also U5.51 (QSPI_SD3)
- net RD+: now also U5.47 (USB_DP)
- net RD-: now also U5.46 (USB_DM)
- net RTCK: now also U5.4 (GPIO2)
- net SWCLK: now also U5.24 (SWCLK)
- net SWDIO: now also U5.25 (SWD)
- net TCK_SWCLK: now also U5.6 (GPIO4)
- net TDI: now also U5.8 (GPIO6)
- net TDO_SWO: now also U5.3 (GPIO1)
- net TMS_SWDIO: now also U5.7 (GPIO5)
- net XIN: now also U5.20 (XIN)
- net ~{SRST}: now also U5.2 (GPIO0)
- net ~{TRST}: now also U5.9 (GPIO7)
- net at J2.15 (~{SRST}), R7.2: now also R20.1
- net at J2.3 (~{TRST}), R6.2: now also R19.1
- net at J2.9 (TCK/SWDCLK), R9.2: now also R21.2
- net at C3.1, R15.2: now also U5.26 (RUN)
- no-connect marks 30 -> 29
Other:
- note added: "RC delay (tau=10(ms))"
- note removed: "RC delay (tau=1(ms))"
- moved on the sheet: C3, R15

Commit message: v2023.07.27
Parts:
- C3: value 0.1uF -> 1uF
- D2: footprint Diode_SMD:D_SOD-323 -> cuhs20s30:US2H
- U2: value W25Q16JVZPIM -> W25Q16JVSNIQ; footprint Package_SON:WSON-8-1EP_6x5mm_P1.27mm_EP3.4x4.3mm -> Package_SO:SO-8_3.9x4.9mm_P1.27mm; MPN W25Q16JVZPIM -> W25Q16JVSNIQ
Changed lines of the file:
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@@
       (effects (font (size 1.27 1.27)))
     )
-    (property "Value" "W25Q16JVZPIM" (at 52.07 118.11 0)
-      (effects (font (size 1.27 1.27)))
-    )
-    (property "Footprint" "Package_SON:WSON-8-1EP_6x5mm_P1.27mm_EP3.4x4.3mm" (at 62.23 105.41 0)
+    (property "Value" "W25Q16JVSNIQ" (at 52.07 118.11 0)
+      (effects (font (size 1.27 1.27)))
+    )
+    (property "Footprint" "Package_SO:SO-8_3.9x4.9mm_P1.27mm" (at 62.23 105.41 0)
       (effects (font (size 1.27 1.27)) hide)
     )
@@
       (effects (font (size 1.27 1.27)) hide)
     )
-    (property "MPN" "W25Q16JVZPIM" (at 62.23 105.41 0)
+    (property "MPN" "W25Q16JVSNIQ" (at 62.23 105.41 0)
       (effects (font (size 1.27 1.27)) hide)
     )
@@
       (effects (font (size 1.27 1.27)) (justify left))
     )
-    (property "Value" "0.1uF" (at 111.76 49.53 0)
+    (property "Value" "1uF" (at 111.76 49.53 0)
       (effects (font (size 1.27 1.27)) (justify left))
     )
@@
       (effects (font (size 1.27 1.27)))
     )
-    (property "Footprint" "Diode_SMD:D_SOD-323" (at 242.57 31.75 0)
-      (effects (font (size 1.27 1.27)) hide)
-    )
+    (property "Footprint" "cuhs20s30:US2H" (at 242.57 31.75 0)
+      (effects (font (size 1.27 1.27)) hide)
+    )

Commit message: update to 2023/09/09 version
Parts:
- D2: value CUHS20S30 -> RB160M-30TR; footprint cuhs20s30:US2H -> pmdu:D_PMDU; MPN CUHS20S30 -> RB160M-30TR
- U2: footprint Package_SO:SO-8_3.9x4.9mm_P1.27mm -> Package_SO:SOIC-8_5.23x5.23mm_P1.27mm; symbol Memory_Flash:W25Q32JVZP -> Memory_Flash:W25Q32JVSS
Connections:
- net GND: no longer U2.9 (EP)
Changed lines of the file:
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@@
   (junction (at 256.54 111.76) (diameter 0) (color 0 0 0 0)
   )
-  (junction (at 62.23 119.38) (diameter 0) (color 0 0 0 0)
-  )
   (junction (at 264.16 111.76) (diameter 0) (color 0 0 0 0)
   )
@@
     (stroke (width 0) (type default))
   )
-  (wire (pts (xy 62.23 118.11) (xy 62.23 119.38))
-    (stroke (width 0) (type default))
-  )
   (wire (pts (xy 166.37 33.02) (xy 166.37 35.56))
     (stroke (width 0) (type default))
@@
     (stroke (width 0) (type default))
   )
-  (wire (pts (xy 64.77 118.11) (xy 64.77 119.38))
-    (stroke (width 0) (type default))
-  )
   (wire (pts (xy 44.45 54.61) (xy 44.45 52.07))
     (stroke (width 0) (type default))
@@
     (stroke (width 0) (type default))
   )
-  (wire (pts (xy 62.23 119.38) (xy 62.23 120.65))
+  (wire (pts (xy 62.23 118.11) (xy 62.23 120.65))
     (stroke (width 0) (type default))
   )
@@
     (stroke (width 0) (type default))
   )
-  (wire (pts (xy 62.23 119.38) (xy 64.77 119.38))
-    (stroke (width 0) (type default))
-  )
   (wire (pts (xy 111.76 165.1) (xy 111.76 171.45))
     (stroke (width 0) (type default))
@@
     )
   )
-  (symbol (lib_id "Memory_Flash:W25Q32JVZP") (at 62.23 105.41 0) (unit 1)
+  (symbol (lib_id "Memory_Flash:W25Q32JVSS") (at 62.23 105.41 0) (unit 1)
     (in_bom yes) (on_board yes) (dnp no)
     (property "Reference" "U2" (at 52.07 115.57 0)
@@
       (effects (font (size 1.27 1.27)))
     )
-    (property "Footprint" "Package_SO:SO-8_3.9x4.9mm_P1.27mm" (at 62.23 105.41 0)
+    (property "Footprint" "Package_SO:SOIC-8_5.23x5.23mm_P1.27mm" (at 62.23 105.41 0)
       (effects (font (size 1.27 1.27)) hide)
     )
-    (property "Datasheet" "http://www.winbond.com/resource-files/w25q32jv%20revg%2003272018%20plus.pdf" (at 62.23 107.95 0)
+    (property "Datasheet" "http://www.winbond.com/resource-files/w25q32jv%20revg%2003272018%20plus.pdf" (at 62.23 105.41 0)
       (effects (font (size 1.27 1.27)) hide)
     )
@@
     (pin "7")
     (pin "8")
-    (pin "9")
     (instances
       (project "rp2040_jtag_debugger"
@@
       (effects (font (size 1.27 1.27)))
     )
-    (property "Value" "CUHS20S30" (at 245.11 29.21 0)
+    (property "Value" "RB160M-30TR" (at 245.11 29.21 0)
       (effects (font (size 1.27 1.27)))
     )
-    (property "Footprint" "cuhs20s30:US2H" (at 242.57 31.75 0)
+    (property "Footprint" "pmdu:D_PMDU" (at 242.57 31.75 0)
       (effects (font (size 1.27 1.27)) hide)
     )
@@
       (effects (font (size 1.27 1.27)) hide)
     )
-    (property "MPN" "CUHS20S30" (at 242.57 31.75 0)
+    (property "MPN" "RB160M-30TR" (at 242.57 31.75 0)
       (effects (font (size 1.27 1.27)) hide)
     )
